File: pcb/gat_blaster_36.kicad_pcb (KiCad board)
At the start: 2 copper layers, 82 parts, among them J1 USB_C_Receptacle_USB2.0, J2 HDMI_A, J3 Conn_01x05_Pin, SW1 SW_Push, SW10 SW_Push, SW11 SW_Push, SW12 SW_Push, SW13 SW_Push, SW14 SW_Push, SW15 SW_Push, SW16 SW_Push, SW17 SW_Push, SW18 SW_Push, SW19 SW_Push, SW2 SW_Push, SW20 SW_Push, SW3 SW_Push, SW4 SW_Push, SW5 SW_Push, SW6 SW_Push, SW7 SW_Push, SW8 SW_Push, SW9 SW_Push, U1 USBLC6-2SC6, U2 TLV1117-33, U3 STM32F072CBTx, Y1 8MHz

Commit message: latest work from len pc
Parts:
- C10, C11, C12, C13, C14, C15, C16, C6, C7, C8, C9, FB2, R10, R11, R12, R13, R14, R15, R16, R17, R18, R5, R6, R7, R9, SW19, SW20, U2, U3, Y1: moved to F.Cu
- J2: moved to B.Cu
- moved C15 140.5 mm to (240.1, 91.4), turned to 0 degrees
- moved C16 140.5 mm to (240.1, 84.6), turned to 180 degrees
- moved Y1 140.5 mm to (240.1, 88.0), turned to 0 degrees
- moved R7 129.7 mm to (234.6, 88.4), turned to 180 degrees
- moved C8 122.2 mm to (230.8, 73.2), turned to 0 degrees
- moved C9 122.1 mm to (230.8, 75.7), turned to 0 degrees
- moved C10 122.1 mm to (230.8, 78.2), turned to 0 degrees
- moved C11 122.1 mm to (230.8, 80.8), turned to 0 degrees
- moved C6 122.1 mm to (230.8, 70.7), turned to 180 degrees
- moved C7 122.1 mm to (230.8, 68.5), turned to 180 degrees
- moved U2 120.9 mm to (230.2, 62.4), turned to 0 degrees
- moved J3 110.3 mm to (195.7, 93.0)
- moved U3 109.8 mm to (224.6, 88.3), turned to 180 degrees
- moved C5 103.8 mm to (190.0, 52.3)
- moved R2 103.8 mm to (193.3, 66.2)
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